Commit message: updated

File: tracer_description/urdf/gazebo.xacro (robot description, xacro)
@@ -6,5 +6,5 @@
     ========================================
 -->
-<robot xmlns:xacro="http://www.ros.org/wiki/xacro">
+<robot xmlns:xacro="http://www.ros.org/wiki/xacro" name="gazebo">
     <gazebo reference="fl_wheel_link">
         <mu1>1</mu1>

File: tracer_description/urdf/ros2_control.xacro (robot description, xacro)
@@ -6,5 +6,5 @@
     ========================================
 -->
-<robot xmlns:xacro="http://www.ros.org/wiki/xacro">
+<robot xmlns:xacro="http://www.ros.org/wiki/xacro" name="ros2_control">
     <ros2_control name="IgnitionSystem" type="system">
         <hardware>
@@ -45,6 +45,6 @@
         <joint name="L_wheel_joint">
             <command_interface name="velocity">
-                <param name="min">-2</param>
-                <param name="max">2</param>
+                <!-- <param name="min">-2</param>
+                <param name="max">2</param> -->
             </command_interface>
             <state_interface name="position"/>
@@ -53,6 +53,6 @@
         <joint name="R_wheel_joint">
             <command_interface name="velocity">
-                <param name="min">-2</param>
-                <param name="max">2</param>
+                <!-- <param name="min">-2</param>
+                <param name="max">2</param> -->
             </command_interface>
             <state_interface name="position"/>
@@ -61,7 +61,8 @@
     </ros2_control>
     <gazebo>
-        <!-- <plugin filename="libignition-gazebo-joint-state-publisher-system.so" name="ignition::gazebo::systems::JointStatePublisher"/> -->
-        <plugin filename="ign_ros2_control-system" name="ign_ros2_control::IgnitionROS2ControlPlugin">
-            <parameters>$(find tracer_ign_sim)/config/tracer_controller_velocity.yaml</parameters>
+        <plugin
+          filename="ign_ros2_control-system"
+          name="ign_ros2_control::IgnitionROS2ControlPlugin">
+          <parameters>$(find tracer_ign_sim)/config/tracer_controller_velocity.yaml</parameters>
         </plugin>
     </gazebo>

File: tracer_description/urdf/tracer_joints.xacro (robot description, xacro)
@@ -6,5 +6,10 @@
     ========================================
 -->
-<robot>
+<robot xmlns:xacro="http://www.ros.org/wiki/xacro" name="tracer joints">
+    <joint name="base_footprint_joint" type="fixed">
+        <parent link="base_footprint"/>
+        <child link="base_link"/>
+        <origin xyz="0 0 0" pry="0 0 0"/>
+    </joint>
     <joint name="base_joint" type="fixed">
         <origin xyz="0 0 0" rpy="0 0 0"/>

File: tracer_description/urdf/tracer_links.xacro (robot description, xacro)
@@ -6,39 +6,40 @@
     ========================================
 -->
-<robot xmlns:xacro="http://www.ros.org/wiki/xacro">
+<robot xmlns:xacro="http://www.ros.org/wiki/xacro" name="tracer links">
     <!-- load meshes -->
     <xacro:macro name="base_link">
-        <mesh filename="file://$(find tracer_ign_sim)/models/tracer/meshes/tracer_base_link_no_wheel.dae"/>
+        <mesh filename="file://$(find tracer_description)/mesh/tracer/meshes/tracer_base_link_no_wheel.dae"/>
     </xacro:macro>
     <xacro:macro name="fl_castor_link">
-        <mesh filename="file://$(find tracer_ign_sim)/models/tracer/meshes/castor_joint.dae"/>
+        <mesh filename="file://$(find tracer_description)/mesh/tracer/meshes/castor_joint.dae"/>
     </xacro:macro>
     <xacro:macro name="fr_castor_link">
-        <mesh filename="file://$(find tracer_ign_sim)/models/tracer/meshes/castor_joint.dae"/>
+        <mesh filename="file://$(find tracer_description)/mesh/tracer/meshes/castor_joint.dae"/>
     </xacro:macro>
     <xacro:macro name="rl_castor_link">
-        <mesh filename="file://$(find tracer_ign_sim)/models/tracer/meshes/castor_joint.dae"/>
+        <mesh filename="file://$(find tracer_description)/mesh/tracer/meshes/castor_joint.dae"/>
     </xacro:macro>
     <xacro:macro name="rr_castor_link">
-        <mesh filename="file://$(find tracer_ign_sim)/models/tracer/meshes/castor_joint.dae"/>
+        <mesh filename="file://$(find tracer_description)/mesh/tracer/meshes/castor_joint.dae"/>
     </xacro:macro>
     <xacro:macro name="fl_wheel_link">
-        <mesh filename="file://$(find tracer_ign_sim)/models/tracer/meshes/castor.dae"/>
+        <mesh filename="file://$(find tracer_description)/mesh/tracer/meshes/castor.dae"/>
     </xacro:macro>
     <xacro:macro name="fr_wheel_link">
-        <mesh filename="file://$(find tracer_ign_sim)/models/tracer/meshes/castor.dae"/>
+        <mesh filename="file://$(find tracer_description)/mesh/tracer/meshes/castor.dae"/>
     </xacro:macro>
     <xacro:macro name="rl_wheel_link">
-        <mesh filename="file://$(find tracer_ign_sim)/models/tracer/meshes/castor.dae"/>
+        <mesh filename="file://$(find tracer_description)/mesh/tracer/meshes/castor.dae"/>
     </xacro:macro>
     <xacro:macro name="rr_wheel_link">
-        <mesh filename="file://$(find tracer_ign_sim)/models/tracer/meshes/castor.dae"/>
+        <mesh filename="file://$(find tracer_description)/mesh/tracer/meshes/castor.dae"/>
     </xacro:macro>
     <xacro:macro name="L_wheel_link">
-        <mesh filename="file://$(find tracer_ign_sim)/models/tracer/meshes/tracer_wheel.dae"/>
+        <mesh filename="file://$(find tracer_description)/mesh/tracer/meshes/tracer_wheel.dae"/>
     </xacro:macro>
     <xacro:macro name="R_wheel_link">
-        <mesh filename="file://$(find tracer_ign_sim)/models/tracer/meshes/tracer_wheel.dae"/>
-    </xacro:macro>
+        <mesh filename="file://$(find tracer_description)/mesh/tracer/meshes/tracer_wheel.dae"/>
+    </xacro:macro>
+    <link name="base_footprint"></link>
     <!-- Initial Link -->
     <link name="inertial_link">
@@ -67,4 +68,10 @@
             </geometry>
         </collision>
+        <sensor name="imu_sensor" type="imu">
+            <always_on>1</always_on>
+            <update_rate>1</update_rate>
+            <visualize>true</visualize>
+            <topic>imu</topic>
+        </sensor>
     </link>
     <!-- ************************************************** -->
